File: schematic.brd (EAGLE design)
At the start: 172.4 x 120.6 mm, 66 parts, among them IC1 74HC541N, IC2 74HC541N, IC3 74HC541N, IC4 74HC541N, J1 61729-1011, U1 EK-TM4C123GXL, U2 MCP23017-E/SP, U3 MCP23017-E/SP, U4 MCP23017-E/SP, U5 MCP23017-E/SP

Commit message: Final version
Parts:
- moved J1 321.5 mm to (130.8, 172.7)
- moved R8 283.6 mm to (132.1, 53.3), turned to 90 degrees
- moved R7 271.7 mm to (129.5, 53.3), turned to 90 degrees
- moved IC4 262.9 mm to (152.4, 137.2), turned to 180 degrees
- moved U2 251.1 mm to (144.8, 151.1), turned to 270 degrees
- moved IC3 240.9 mm to (135.9, 40.6)
- moved R27 238.2 mm to (156.2, 124.5), turned to 90 degrees
- moved R36 237.5 mm to (167.6, 69.8), turned to 90 degrees
- moved R26 230.5 mm to (158.8, 125.7), turned to 270 degrees
- moved R13 228.9 mm to (144.8, 53.3), turned to 90 degrees
- moved R35 223.8 mm to (162.6, 69.8), turned to 90 degrees
- moved R37 218.2 mm to (94.0, 12.7), turned to 270 degrees
- moved R12 217.7 mm to (142.2, 53.3), turned to 90 degrees
- moved R20 215.8 mm to (64.8, 64.8), turned to 180 degrees
- moved R25 215.7 mm to (153.7, 124.5), turned to 270 degrees
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Connections:
- removed net +5V: IC1.20, IC2.20, IC3.20, IC4.20, J1.1
- removed net N$84: U5.4
- removed net N$85: U5.3
- removed net N$86: U5.2
- removed net N$94: IC1.1, IC1.19, IC2.1, IC2.19, IC3.1, IC3.19, IC4.1, IC4.19, R1.3, R2.3, R37.1, R38.1, U1.J2_1, U1.J3_2, U2.10, U2.15, U2.16, U3.10, U3.16, U3.17, U4.10, U4.15, U4.16, U4.17, U5.10, U5.15, U5.17
- new net N$42: IC1.20, IC2.20, IC3.20, IC4.20, J1.1, R1.1, R2.1, R3.2, R4.2, R5.2, R6.2
- net 0: now also IC1.1, IC1.19, IC2.1, IC2.19, IC3.1, IC3.19, IC4.1, IC4.19, R1.3, R2.3, R37.1, R38.1, S3.3, S4.3, S5.3, S6.3, U1.J2_1, U1.J3_2, U2.10, U2.15, U2.16, U3.10, U3.16, U3.17, U4.10, U4.15, U4.16, U4.17, U5.10, U5.15, U5.17
- net N$104: no longer R1.1, R2.1, R3.2, R4.2, R5.2, R6.2
- net N$87: now also S3.2; no longer S3.3
- net N$88: now also S4.2; no longer S4.3
- net N$89: now also S5.2; no longer S5.3
- net N$90: now also S6.2; no longer S6.3
Routing:
- net 0: track 0.00 -> 702.8 mm
- net N$104: track 0.00 -> 488.1 mm
- net N$42: track 0.00 -> 479.6 mm
- net N$102: track 0.00 -> 377.0 mm, vias 0 -> 1
- net N$103: track 0.00 -> 369.7 mm
- net N$98: track 0.00 -> 211.5 mm
- net N$99: track 0.00 -> 179.0 mm
- net N$87: track 0.00 -> 175.7 mm, vias 0 -> 1
- net N$90: track 0.00 -> 159.1 mm
- net N$100: track 0.00 -> 155.6 mm
- net N$89: track 0.00 -> 155.0 mm, vias 0 -> 1
- net N$101: track 0.00 -> 154.0 mm, vias 0 -> 1
- net N$88: track 0.00 -> 152.2 mm, vias 0 -> 1
- net N$131: track 0.00 -> 113.3 mm
- net N$121: track 0.00 -> 108.2 mm
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Other:
- board size 172.4 x 120.6 mm -> 171.1 x 179.1 mm
- board text added: "C:/Users/DIYGary/Documents/Projects/Hardware/InstrumentPanel/diygarylogo_B.bmp"
