File: schematic.sch (EAGLE design)
At the start: 27 parts, among them U1 EK-TM4C123GXL, U2 MCP23017-E/SP, U3 MCP23017-E/SP, U4 MCP23017-E/SP, U5 MCP23017-E/SP

Commit message: Update schematic.sch
Parts:
- added IC1, IC2, IC3, IC4: 74HC541N, 74xx-eu:74HC541N
Connections:
- new net N$1: IC1A.A8, U4.GPA0
- new net N$10: IC1A.A6, U4.GPA2
- new net N$11: IC1A.A5, U4.GPA3
- new net N$12: IC1A.A4, U4.GPA4
- new net N$13: IC1A.A3, U4.GPA5
- new net N$14: IC1A.A2, U4.GPA6
- new net N$15: IC1A.A1, U4.GPA7
- new net N$16: LED8.COM@1, U4.GPB7
- new net N$17: LED1.CA@1, U4.GPB6
- new net N$18: LED1.CA@2, U4.GPB5
- new net N$19: LED1.CA@3, U4.GPB4
- new net N$2: IC1A.Y2, LED1.B, LED6.B, LED8.B
- new net N$3: IC1A.Y3, LED1.C, LED6.C, LED8.C
- new net N$4: IC1A.Y4, LED1.D, LED6.D, LED8.D
- new net N$5: IC1A.Y5, LED1.E, LED6.E, LED8.E
- new net N$6: IC1A.Y6, LED1.F, LED6.F, LED8.F
- new net N$7: IC1A.Y7, LED1.G, LED6.G, LED8.G
- new net N$8: IC1A.Y1, LED1.A, LED6.A, LED8.A
- new net N$9: IC1A.A7, U4.GPA1
Other:
- moved on the sheet: LED1, LED2, LED3, LED4, LED5, LED6, LED7, LED8, U2, U3, U4, U5

Commit message: Update schematic.sch
Parts:
- removed LED12, LED13: TLLY4400, led:TLLY4400
Connections:
- new net N$20: IC4A.Y1, LED2.A, LED5.A, LED7.A
- new net N$21: IC4A.Y2, LED2.B, LED5.B, LED7.B
- new net N$22: IC4A.Y3, LED2.C, LED5.C, LED7.C
- new net N$23: IC4A.Y4, LED2.D, LED5.D, LED7.D
- new net N$24: IC4A.Y5, LED2.E, LED5.E, LED7.E
- new net N$25: IC4A.Y6, LED2.F, LED5.F, LED7.F
- new net N$26: IC4A.Y7, LED2.G, LED5.G, LED7.G
- new net N$27: IC4A.Y8, LED2.DP
- new net N$28: IC1A.Y8, LED1.DP
- new net N$29: LED2.CA@2, U2.GPB4
- new net N$30: LED5.COM@1, U2.GPB6
- new net N$31: LED2.CA@1, U2.GPB5
- new net N$32: LED2.CA@3, U2.GPB3
- new net N$33: IC4A.A8, U2.GPA0
- new net N$34: IC4A.A7, U2.GPA1
- new net N$35: IC4A.A6, U2.GPA2
- new net N$36: IC4A.A5, U2.GPA3
- new net N$37: IC4A.A4, U2.GPA4
- new net N$38: IC4A.A3, U2.GPA5
- new net N$39: IC4A.A2, U2.GPA6
- new net N$40: IC4A.A1, U2.GPA7
- new net N$41: IC3A.Y1, LED4.A
- new net N$42: IC3A.Y2, LED4.B
- new net N$43: IC3A.Y3, LED4.C
- new net N$44: IC3A.Y4, LED4.D
- new net N$45: IC3A.Y5, LED4.E
- new net N$46: IC3A.Y6, LED4.F
- new net N$47: IC3A.Y7, LED4.G
- new net N$48: IC3A.Y8, LED4.DP
- new net N$49: LED4.CA@1, U5.GPB7
- new net N$50: LED4.CA@2, U5.GPB6
- new net N$51: LED4.CA@3, U5.GPB5
- new net N$52: IC3A.A1, U5.GPA7
- new net N$53: IC3A.A2, U5.GPA6
- new net N$54: IC3A.A3, U5.GPA5
- new net N$55: IC3A.A4, U5.GPA4
- new net N$56: IC3A.A5, U5.GPA3
- new net N$57: IC3A.A6, U5.GPA2
- new net N$58: IC3A.A7, U5.GPA1
- new net N$59: IC3A.A8, U5.GPA0
- new net N$60: IC2A.A1, U3.GPA7
- new net N$61: IC2A.A2, U3.GPA6
- new net N$62: IC2A.A3, U3.GPA5
- new net N$63: IC2A.A4, U3.GPA4
- new net N$64: IC2A.A5, U3.GPA3
- new net N$65: IC2A.A6, U3.GPA2
- new net N$66: IC2A.A7, U3.GPA1
- new net N$67: IC2A.A8, U3.GPA0
- new net N$68: IC2A.Y1, LED3.A
- new net N$69: IC2A.Y2, LED3.B
- new net N$70: IC2A.Y3, LED3.C
- new net N$71: IC2A.Y4, LED3.D
- new net N$72: IC2A.Y5, LED3.E
- new net N$73: IC2A.Y6, LED3.F
- new net N$74: IC2A.Y7, LED3.G
- new net N$75: IC2A.Y8, LED3.DP
- new net N$76: LED3.CA@1, U3.GPB7
- new net N$77: LED3.CA@2, U3.GPB6
- new net N$78: LED3.CA@3, U3.GPB5
- new net N$79: U1.GND, U2.A0, U2.A1, U3.A1, U3.A2, U4.A0, U4.A1, U4.A2, U5.A0, U5.A2
- new net N$80: LED7.COM@2, U2.GPB7
- new net N$81: LED10.C, LED11.C, LED14.C, LED9.C, U1.+3.3V, U2.A2, U2.VDD, U3.A0, U3.VDD, U4.VDD, U5.A1, U5.VDD
- new net N$82: LED6.COM@2, U4.GPB7
- new net N$83: LED9.A, S3.O, U5.GPB4
- new net N$84: LED10.A, S4.O, U5.GPB3
- new net N$85: LED11.A, S5.O, U5.GPB2
- new net N$86: LED14.A, S6.O, U5.GPB1
- new net N$87: S3.S, U1.PE5
- new net N$88: S4.S, U1.PE4
- new net N$89: S5.S, U1.PE3
- new net N$90: S6.S, U1.PE2
- net N$16: now also U4.GPB6; no longer U4.GPB7
- net N$17: now also U4.GPB5; no longer U4.GPB6
- net N$18: now also U4.GPB4; no longer U4.GPB5
- net N$19: now also U4.GPB3; no longer U4.GPB4
Other:
- moved on the sheet: IC2, IC3, LED10, LED11, LED14, LED3, LED4, LED5, LED7, LED9, S3, S4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

Commit message: Update schematic.sch
Parts:
- added R3, R4, R5, R6: (no value), rcl:R-US_0204/7
Connections:
- removed net N$81: LED10.C, LED11.C, LED14.C, LED9.C, U1.+3.3V, U2.A2, U2.VDD, U3.A0, U3.VDD, U4.VDD, U5.A1, U5.VDD
- new net +5V: IC1P.VCC, IC2P.VCC, IC3P.VCC, IC4P.VCC
- new net 0: IC1P.GND, IC2P.GND, IC3P.GND, IC4P.GND
- new net N$100: R1.S, U1.PB4
- new net N$101: R2.S, U1.PB5
- new net N$102: U1.PB2, U2.SCL, U3.SCL, U4.SCL, U5.SCL
- new net N$103: U1.PB3, U2.SDA, U3.SDA, U4.SDA, U5.SDA
- new net N$104: R1.A, R2.A, R3.2, R4.2, R5.2, R6.2, S1.P, S2.S1, U1.+3.3V, U2.!RESET, U2.A2, U2.VDD, U3.!RESET, U3.A0, U3.VDD, U4.!RESET, U4.VDD, U5.!RESET, U5.A1, U5.VDD
- new net N$91: LED14.A, R3.1
- new net N$92: LED11.C, S5.O
- new net N$93: LED11.A, R4.1
- new net N$94: IC1A.G1, IC1A.G2, IC2A.G1, IC2A.G2, IC3A.G1, IC3A.G2, IC4A.G1, IC4A.G2, R1.E, R2.E, S1.P1, S2.S, U1.GND, U2.A0, U2.A1, U2.VSS, U3.A1, U3.A2, U3.VSS, U4.A0, U4.A1, U4.A2, U4.VSS, U5.A0, U5.A2, U5.VSS
- new net N$95: LED9.C, S3.O
- new net N$96: LED10.A, R5.1
- new net N$97: LED9.A, R6.1
- new net N$98: S2.P, S2.P1, U1.PE1
- new net N$99: S1.S, S1.S1, U1.PE0
- net N$79: now also LED14.C, S6.O; no longer U1.GND, U2.A0, U2.A1, U3.A1, U3.A2, U4.A0, U4.A1, U4.A2, U5.A0, U5.A2
- net N$83: now also LED10.C, S4.O; no longer LED9.A, S3.O, U5.GPB4
- net N$84: no longer LED10.A, S4.O
- net N$85: no longer LED11.A, S5.O
- net N$86: no longer LED14.A, S6.O
Other:
- moved on the sheet: LED10, LED11, LED14, LED9, R1, R2, S1, S2, S5, S6

Commit message: Update schematic.sch
Parts:
- added R10, R11, R12, R13, R14, R15, R16, R17, R18, R19, R20, R21, R22, R23, R24, R25, R26, R27, R28, R29, R30, R31, R32, R33, R34, R7, R8, R9: (no value), rcl:R-US_0204/7
Connections:
- removed net N$2: IC1A.Y2, LED1.B, LED6.B, LED8.B
- removed net N$3: IC1A.Y3, LED1.C, LED6.C, LED8.C
- removed net N$4: IC1A.Y4, LED1.D, LED6.D, LED8.D
- removed net N$5: IC1A.Y5, LED1.E, LED6.E, LED8.E
- removed net N$6: IC1A.Y6, LED1.F, LED6.F, LED8.F
- removed net N$7: IC1A.Y7, LED1.G, LED6.G, LED8.G
- new net N$105: IC2A.Y6, R19.1
- new net N$106: LED3.E, R18.2
- new net N$107: IC2A.Y4, R17.1
- new net N$108: LED3.C, R16.2
- new net N$109: IC2A.Y2, R15.1
- new net N$110: LED3.A, R14.2
- new net N$111: LED4.G, R13.2
- new net N$112: IC3A.Y6, R12.1
- new net N$113: LED4.E, R11.2
- new net N$114: IC3A.Y4, R10.1
- new net N$115: LED4.C, R9.2
- new net N$116: IC3A.Y2, R8.1
- new net N$117: LED4.A, R7.2
- new net N$118: IC1A.Y1, R33.2
- new net N$119: LED2.B, LED5.B, LED7.B, R27.1
- new net N$120: LED2.C, LED5.C, LED7.C, R25.2
- new net N$121: LED2.D, LED5.D, LED7.D, R24.2
- new net N$123: LED2.F, LED5.F, LED7.F, R22.2
- new net N$124: LED2.G, LED5.G, LED7.G, R21.2
- new net N$125: IC1A.Y2, R34.2
- new net N$126: LED1.B, LED6.B, LED8.B, R34.1
- new net N$127: LED1.C, LED6.C, LED8.C, R32.2
- new net N$128: LED1.D, LED6.D, LED8.D, R31.2
- new net N$129: LED1.E, LED6.E, LED8.E, R30.2
- new net N$130: LED1.F, LED6.F, LED8.F, R29.2
- new net N$131: LED1.G, LED6.G, LED8.G, R28.2
- new net N$132: IC4A.Y3, R25.1
- new net N$133: IC4A.Y4, R24.1
- new net N$134: IC4A.Y5, R23.1
- new net N$135: IC4A.Y6, R22.1
- new net N$136: IC4A.Y7, R21.1
- new net N$137: IC4A.Y1, R26.1
- new net N$138: IC4A.Y2, R27.2
- new net N$81: LED3.G, R20.2
- net N$20: now also R26.2; no longer IC4A.Y1
- net N$21: now also IC1A.Y3, R32.1; no longer IC4A.Y2, LED2.B, LED5.B, LED7.B
- net N$22: now also IC1A.Y7, R28.1; no longer IC4A.Y3, LED2.C, LED5.C, LED7.C
- net N$23: now also IC1A.Y6, R29.1; no longer IC4A.Y4, LED2.D, LED5.D, LED7.D
- net N$24: now also R23.2; no longer IC4A.Y5
- net N$25: now also IC1A.Y5, R30.1; no longer IC4A.Y6, LED2.F, LED5.F, LED7.F
- net N$26: now also IC1A.Y4, R31.1; no longer IC4A.Y7, LED2.G, LED5.G, LED7.G
- net N$41: now also R7.1; no longer LED4.A
- net N$42: now also R8.2; no longer IC3A.Y2
- net N$43: now also R9.1; no longer LED4.C
- net N$44: now also R10.2; no longer IC3A.Y4
- net N$45: now also R11.1; no longer LED4.E
- net N$46: now also R12.2; no longer IC3A.Y6
- net N$47: now also R13.1; no longer LED4.G
- net N$68: now also R14.1; no longer LED3.A
- net N$69: now also R15.2; no longer IC2A.Y2
- net N$70: now also R16.1; no longer LED3.C
- net N$71: now also R17.2; no longer IC2A.Y4
- net N$72: now also R18.1; no longer LED3.E
- net N$73: now also R19.2; no longer IC2A.Y6
- net N$74: now also R20.1; no longer LED3.G
- net N$8: now also R33.1; no longer IC1A.Y1

Commit message: Update schematic.sch
Parts:
- added R35, R36, R37, R38: (no value), rcl:R-US_0204/7
Connections:
- net N$102: now also R35.1
- net N$103: now also R36.1
- net N$104: now also R35.2, R36.2
- net N$94: now also R37.1, R38.1; no longer S1.P1, S2.S
- net N$98: now also R38.2
- net N$99: now also R37.2
Other:
- note added: "Gary T Smith / DIYGary"
Changed lines of the file:
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@@
 <part name="R33" library="rcl" library_urn="urn:adsk.eagle:library:334" deviceset="R-US_" device="0204/7" package3d_urn="urn:adsk.eagle:package:23498/2"/>
 <part name="R34" library="rcl" library_urn="urn:adsk.eagle:library:334" deviceset="R-US_" device="0204/7" package3d_urn="urn:adsk.eagle:package:23498/2"/>
+<part name="R35" library="rcl" library_urn="urn:adsk.eagle:library:334" deviceset="R-US_" device="0204/7" package3d_urn="urn:adsk.eagle:package:23498/2"/>
+<part name="R36" library="rcl" library_urn="urn:adsk.eagle:library:334" deviceset="R-US_" device="0204/7" package3d_urn="urn:adsk.eagle:package:23498/2"/>
+<part name="R37" library="rcl" library_urn="urn:adsk.eagle:library:334" deviceset="R-US_" device="0204/7" package3d_urn="urn:adsk.eagle:package:23498/2"/>
+<part name="R38" library="rcl" library_urn="urn:adsk.eagle:library:334" deviceset="R-US_" device="0204/7" package3d_urn="urn:adsk.eagle:package:23498/2"/>
 </parts>
 <sheets>
 <sheet>
 <plain>
+<text x="60.96" y="22.86" size="1.778" layer="91">Gary T Smith / DIYGary</text>
 </plain>
 <instances>
@@
 <attribute name="NAME" x="189.23" y="115.7986" size="1.778" layer="95"/>
 <attribute name="VALUE" x="189.23" y="110.998" size="1.778" layer="96"/>
+</instance>
+<instance part="R35" gate="G$1" x="38.1" y="-187.96" smashed="yes">
+<attribute name="NAME" x="34.29" y="-186.4614" size="1.778" layer="95"/>
+<attribute name="VALUE" x="34.29" y="-191.262" size="1.778" layer="96"/>
+</instance>
+<instance part="R36" gate="G$1" x="38.1" y="-180.34" smashed="yes">
+<attribute name="NAME" x="34.29" y="-178.8414" size="1.778" layer="95"/>
+<attribute name="VALUE" x="34.29" y="-183.642" size="1.778" layer="96"/>
+</instance>
+<instance part="R37" gate="G$1" x="-40.64" y="-43.18" smashed="yes" rot="R90">
+<attribute name="NAME" x="-42.1386" y="-46.99" size="1.778" layer="95" rot="R90"/>
+<attribute name="VALUE" x="-37.338" y="-46.99" size="1.778" layer="96" rot="R90"/>
+</instance>
+<instance part="R38" gate="G$1" x="-35.56" y="-43.18" smashed="yes" rot="R90">
+<attribute name="NAME" x="-37.0586" y="-46.99" size="1.778" layer="95" rot="R90"/>
+<attribute name="VALUE" x="-32.258" y="-46.99" size="1.778" layer="96" rot="R90"/>
 </instance>
 </instances>
@@
 <wire x1="96.52" y1="-139.7" x2="53.34" y2="-139.7" width="0.1524" layer="91"/>
 <junction x="53.34" y="-139.7"/>
-<pinref part="S1" gate="1" pin="P1"/>
-<wire x1="-53.34" y1="-25.4" x2="-55.88" y2="-25.4" width="0.1524" layer="91"/>
-<wire x1="-55.88" y1="-25.4" x2="-55.88" y2="-30.48" width="0.1524" layer="91"/>
-<wire x1="-55.88" y1="-30.48" x2="-55.88" y2="-213.36" width="0.1524" layer="91"/>
-<wire x1="-55.88" y1="-213.36" x2="53.34" y2="-213.36" width="0.1524" layer="91"/>
 <junction x="53.34" y="-213.36"/>
-<pinref part="S2" gate="1" pin="S"/>
-<wire x1="-53.34" y1="-30.48" x2="-55.88" y2="-30.48" width="0.1524" layer="91"/>
-<junction x="-55.88" y="-30.48"/>
 <pinref part="R1" gate="G$1" pin="E"/>
+<wire x1="-35.56" y1="-213.36" x2="53.34" y2="-213.36" width="0.1524" layer="91"/>
 <wire x1="22.86" y1="48.26" x2="53.34" y2="48.26" width="0.1524" layer="91"/>
 <junction x="53.34" y="48.26"/>
@@
 <wire x1="22.86" y1="66.04" x2="53.34" y2="66.04" width="0.1524" layer="91"/>
 <junction x="53.34" y="66.04"/>
+<pinref part="R37" gate="G$1" pin="1"/>
+<wire x1="-40.64" y1="-48.26" x2="-40.64" y2="-213.36" width="0.1524" layer="91"/>
+<wire x1="-40.64" y1="-213.36" x2="-35.56" y2="-213.36" width="0.1524" layer="91"/>
+<pinref part="R38" gate="G$1" pin="1"/>
+<wire x1="-35.56" y1="-48.26" x2="-35.56" y2="-213.36" width="0.1524" layer="91"/>
+<junction x="-35.56" y="-213.36"/>
 </segment>
 </net>
@@
 <pinref part="S2" gate="1" pin="P1"/>
 <pinref part="U1" gate="G$1" pin="PE1"/>
-<wire x1="-43.18" y1="-27.94" x2="-17.78" y2="-27.94" width="0.1524" layer="91"/>
+<wire x1="-43.18" y1="-27.94" x2="-35.56" y2="-27.94" width="0.1524" layer="91"/>
 <pinref part="S2" gate="1" pin="P"/>
+<wire x1="-35.56" y1="-27.94" x2="-17.78" y2="-27.94" width="0.1524" layer="91"/>
 <wire x1="-43.18" y1="-27.94" x2="-43.18" y2="-30.48" width="0.1524" layer="91"/>
 <junction x="-43.18" y="-27.94"/>
+<wire x1="-35.56" y1="-27.94" x2="-35.56" y2="-38.1" width="0.1524" layer="91"/>
+<junction x="-35.56" y="-27.94"/>
+<pinref part="R38" gate="G$1" pin="2"/>
 </segment>
 </net>
@@
 <pinref part="S1" gate="1" pin="S1"/>
 <pinref part="U1" gate="G$1" pin="PE0"/>
-<wire x1="-43.18" y1="-25.4" x2="-17.78" y2="-25.4" width="0.1524" layer="91"/>
+<wire x1="-43.18" y1="-25.4" x2="-40.64" y2="-25.4" width="0.1524" layer="91"/>
 <pinref part="S1" gate="1" pin="S"/>
+<wire x1="-40.64" y1="-25.4" x2="-17.78" y2="-25.4" width="0.1524" layer="91"/>
 <wire x1="-43.18" y1="-22.86" x2="-43.18" y2="-25.4" width="0.1524" layer="91"/>
 <junction x="-43.18" y="-25.4"/>
+<wire x1="-40.64" y1="-25.4" x2="-40.64" y2="-38.1" width="0.1524" layer="91"/>
+<junction x="-40.64" y="-25.4"/>
+<pinref part="R37" gate="G$1" pin="2"/>
 </segment>
 </net>
@@
 <wire x1="129.54" y1="-180.34" x2="129.54" y2="-198.12" width="0.1524" layer="91"/>
 <wire x1="129.54" y1="-198.12" x2="48.26" y2="-198.12" width="0.1524" layer="91"/>
-<wire x1="48.26" y1="-198.12" x2="48.26" y2="-106.68" width="0.1524" layer="91"/>
+<wire x1="48.26" y1="-198.12" x2="48.26" y2="-185.42" width="0.1524" layer="91"/>
 <junction x="48.26" y="-106.68"/>
+<pinref part="R35" gate="G$1" pin="1"/>
+<wire x1="48.26" y1="-185.42" x2="48.26" y2="-106.68" width="0.1524" layer="91"/>
+<wire x1="33.02" y1="-187.96" x2="33.02" y2="-185.42" width="0.1524" layer="91"/>
+<wire x1="33.02" y1="-185.42" x2="48.26" y2="-185.42" width="0.1524" layer="91"/>
+<junction x="48.26" y="-185.42"/>
 </segment>
 </net>
@@
 <wire x1="132.08" y1="-177.8" x2="132.08" y2="-200.66" width="0.1524" layer="91"/>
 <wire x1="132.08" y1="-200.66" x2="45.72" y2="-200.66" width="0.1524" layer="91"/>
-<wire x1="45.72" y1="-200.66" x2="45.72" y2="-111.76" width="0.1524" layer="91"/>
+<wire x1="45.72" y1="-200.66" x2="45.72" y2="-182.88" width="0.1524" layer="91"/>
 <junction x="45.72" y="-111.76"/>
+<pinref part="R36" gate="G$1" pin="1"/>
+<wire x1="45.72" y1="-182.88" x2="45.72" y2="-111.76" width="0.1524" layer="91"/>
+<wire x1="33.02" y1="-180.34" x2="33.02" y2="-182.88" width="0.1524" layer="91"/>
+<wire x1="33.02" y1="-182.88" x2="45.72" y2="-182.88" width="0.1524" layer="91"/>
+<junction x="45.72" y="-182.88"/>
 </segment>
 </net>
@@
 <pinref part="U3" gate="G$1" pin="VDD"/>
 <wire x1="50.8" y1="-101.6" x2="50.8" y2="-109.22" width="0.1524" layer="91"/>
-<wire x1="50.8" y1="-109.22" x2="50.8" y2="-190.5" width="0.1524" layer="91"/>
+<wire x1="50.8" y1="-109.22" x2="50.8" y2="-180.34" width="0.1524" layer="91"/>
+<wire x1="50.8" y1="-180.34" x2="50.8" y2="-187.96" width="0.1524" layer="91"/>
+<wire x1="50.8" y1="-187.96" x2="50.8" y2="-190.5" width="0.1524" layer="91"/>
 <wire x1="50.8" y1="-190.5" x2="83.82" y2="-190.5" width="0.1524" layer="91"/>
 <junction x="50.8" y="-101.6"/>
@@
 <wire x1="93.98" y1="-203.2" x2="93.98" y2="-190.5" width="0.1524" layer="91"/>
 <junction x="93.98" y="-190.5"/>
-</segment>
-</net>
+<wire x1="50.8" y1="-187.96" x2="43.18" y2="-187.96" width="0.1524" layer="91"/>
+<junction x="50.8" y="-187.96"/>
+<pinref part="R35" gate="G$1" pin="2"/>
+<pinref part="R36" gate="G$1" pin="2"/>
+<wire x1="43.18" y1="-180.34" x2="50.8" y2="-180.34" width="0.1524" layer="91"/>
+<junction x="50.8" y="-180.34"/>
+</segment>
+</net>

Commit message: Schematic finished, board partially done
Parts:
- removed LED1, LED2, LED3, LED4: BA56-12EWA, display-kingbright:BA56-12EWA
- removed LED5, LED6, LED7, LED8: 7-SEG_SA10-21, display-kingbright:7-SEG_SA10-21
- added D1, D2, D3, D4: (no value), 5611AH:5611AH
- added DS1, DS2, DS3, DS4: 5631AH, 5631AH:5631AH
- added J1: 61729-1011, Connector_USB:61729-1011
Connections:
- removed net N$42: LED4.B, R8.2
- removed net N$44: LED4.D, R10.2
- removed net N$46: LED4.F, R12.2
- removed net N$69: LED3.B, R15.2
- removed net N$71: LED3.D, R17.2
- removed net N$73: LED3.F, R19.2
- new net N$2: DS1.A_B, R15.2
- new net N$3: DS1.A_D, R17.2
- new net N$4: DS1.A_F, R19.2
- new net N$5: DS2.A_B, R8.2
- new net N$6: DS2.A_D, R10.2
- new net N$7: DS2.A_F, R12.2
- net +5V: now also J1.VCC
- net 0: now also J1.GND
- net N$106: now also DS1.A_E; no longer LED3.E
- net N$108: now also DS1.A_C; no longer LED3.C
- net N$110: now also DS1.A_A; no longer LED3.A
- net N$111: now also DS2.A_G; no longer LED4.G
- net N$113: now also DS2.A_E; no longer LED4.E
- net N$115: now also DS2.A_C; no longer LED4.C
- net N$117: now also DS2.A_A; no longer LED4.A
- net N$119: now also D1.B, D2.B, DS3.A_B; no longer LED2.B, LED5.B, LED7.B
- net N$120: now also D1.C, D2.C, DS3.A_C; no longer LED2.C, LED5.C, LED7.C
- net N$121: now also D1.D, D2.D, DS3.A_D; no longer LED2.D, LED5.D, LED7.D
- net N$123: now also D1.F, D2.F, DS3.A_F; no longer LED2.F, LED5.F, LED7.F
- net N$124: now also D1.G, D2.G, DS3.A_G; no longer LED2.G, LED5.G, LED7.G
- net N$126: now also D3.B, D4.B, DS4.A_B; no longer LED1.B, LED6.B, LED8.B
- net N$127: now also D3.C, D4.C, DS4.A_C; no longer LED1.C, LED6.C, LED8.C
- net N$128: now also D3.D, D4.D, DS4.A_D; no longer LED1.D, LED6.D, LED8.D
- net N$129: now also D3.E, D4.E, DS4.A_E; no longer LED1.E, LED6.E, LED8.E
- net N$130: now also D3.F, D4.F, DS4.A_F; no longer LED1.F, LED6.F, LED8.F
- net N$131: now also D3.G, D4.G, DS4.A_G; no longer LED1.G, LED6.G, LED8.G
- net N$16: now also D3.CK1; no longer LED8.COM@1
- net N$17: now also DS4.CC_D1; no longer LED1.CA@1
- net N$18: now also DS4.CC_D2; no longer LED1.CA@2
- net N$19: now also DS4.CC_D3; no longer LED1.CA@3
- net N$20: now also D1.A, D2.A, DS3.A_A; no longer LED2.A, LED5.A, LED7.A
- net N$24: now also D1.E, D2.E, DS3.A_E; no longer LED2.E, LED5.E, LED7.E
- net N$27: now also DS3.A_DP; no longer LED2.DP
- net N$28: now also DS4.A_DP; no longer LED1.DP
- net N$29: now also DS3.CC_D2; no longer LED2.CA@2
- net N$30: now also D1.CK1; no longer LED5.COM@1
- net N$31: now also DS3.CC_D1; no longer LED2.CA@1
- net N$32: now also DS3.CC_D3; no longer LED2.CA@3
- net N$48: now also DS2.A_DP; no longer LED4.DP
- net N$49: now also DS2.CC_D1; no longer LED4.CA@1
- net N$50: now also DS2.CC_D2; no longer LED4.CA@2
- net N$51: now also DS2.CC_D3; no longer LED4.CA@3
- net N$75: now also DS1.A_DP; no longer LED3.DP
- net N$76: now also DS1.CC_D1; no longer LED3.CA@1
- net N$77: now also DS1.CC_D2; no longer LED3.CA@2
- net N$78: now also DS1.CC_D3; no longer LED3.CA@3
- net N$8: now also D3.A, D4.A, DS4.A_A; no longer LED1.A, LED6.A, LED8.A
- net N$80: now also D2.CK2; no longer LED7.COM@2
- net N$81: now also DS1.A_G; no longer LED3.G
- net N$82: now also D4.CK2; no longer LED6.COM@2

Commit message: Final version
Connections:
- removed net +5V: IC1P.VCC, IC2P.VCC, IC3P.VCC, IC4P.VCC, J1.VCC
- removed net N$84: U5.GPB3
- removed net N$85: U5.GPB2
- removed net N$86: U5.GPB1
- removed net N$94: IC1A.G1, IC1A.G2, IC2A.G1, IC2A.G2, IC3A.G1, IC3A.G2, IC4A.G1, IC4A.G2, R1.E, R2.E, R37.1, R38.1, U1.GND, U2.A0, U2.A1, U2.VSS, U3.A1, U3.A2, U3.VSS, U4.A0, U4.A1, U4.A2, U4.VSS, U5.A0, U5.A2, U5.VSS
- new net N$42: IC1P.VCC, IC2P.VCC, IC3P.VCC, IC4P.VCC, J1.VCC, R1.A, R2.A, R3.2, R4.2, R5.2, R6.2
- net 0: now also IC1A.G1, IC1A.G2, IC2A.G1, IC2A.G2, IC3A.G1, IC3A.G2, IC4A.G1, IC4A.G2, R1.E, R2.E, R37.1, R38.1, S3.S, S4.S, S5.S, S6.S, U1.GND, U2.A0, U2.A1, U2.VSS, U3.A1, U3.A2, U3.VSS, U4.A0, U4.A1, U4.A2, U4.VSS, U5.A0, U5.A2, U5.VSS
- net N$104: no longer R1.A, R2.A, R3.2, R4.2, R5.2, R6.2
- net N$87: now also S3.P; no longer S3.S
- net N$88: now also S4.P; no longer S4.S
- net N$89: now also S5.P; no longer S5.S
- net N$90: now also S6.P; no longer S6.S
